File: eagle/aWXIrons/main.brd (EAGLE design)
At the start: 182 x 40 mm, 52 parts, among them IC1_DUAL OPA336U, IC1_SINGLE OPA336U, Q1 BSN20, Q2 BSN20

Commit message: Change +12V to +9V in schematic and PCBs. Update PDFs.
Connections:
- net +12V renamed +9V
Routing:
- net +9V: track 117.9 -> 96.6 mm
Other:
- board text added: "aWXIron v1.2.1"
- board text removed: "aWXIron v1.2"
Changed lines of the file:
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@@
 <wire x1="57.785" y1="35.8775" x2="57.785" y2="28.8925" width="0.4064" layer="42" style="dashdot"/>
 <wire x1="57.785" y1="28.8925" x2="56.1975" y2="28.8925" width="0.4064" layer="42" style="dashdot"/>
-<text x="77.47" y="30.1625" size="1.778" layer="1" ratio="15">aWXIron v1.2</text>
+<text x="76.454" y="30.1625" size="1.778" layer="1" ratio="15">aWXIron v1.2.1</text>
 <text x="76.835" y="27.305" size="1.778" layer="1" ratio="15">F1RMB - 2015</text>
 <rectangle x1="75.565" y1="26.3525" x2="97.155" y2="32.7025" layer="41"/>
 <rectangle x1="20.2565" y1="28.8925" x2="25.4" y2="30.353" layer="17"/>
 <rectangle x1="50.673" y1="29.21" x2="56.007" y2="30.7975" layer="17"/>
+<rectangle x1="23.749" y1="33.909" x2="27.051" y2="35.56" layer="17"/>
+<rectangle x1="54.102" y1="33.909" x2="57.404" y2="35.56" layer="17"/>
 </plain>
 <attributes>
@@
 <wire x1="21.59" y1="26.9875" x2="27.7925" y2="26.9875" width="0.4064" layer="16"/>
 </signal>
-<signal name="+12V">
-<contactref element="R3" pad="2"/>
-<contactref element="R4" pad="2"/>
-<contactref element="U$3" pad="1"/>
-<contactref element="U$3" pad="3"/>
-<contactref element="U$3" pad="2"/>
-<contactref element="U$2" pad="3"/>
-<contactref element="U$2" pad="1"/>
-<contactref element="U$2" pad="2"/>
-<contactref element="U$1" pad="VIN"/>
-<contactref element="JP_12V" pad="1"/>
-<wire x1="43.18" y1="23.705825" x2="24.6888625" y2="23.705825" width="0.6096" layer="16"/>
-<wire x1="43.18" y1="35.56" x2="43.18" y2="24.4475" width="0.6096" layer="16"/>
-<wire x1="43.18" y1="24.4475" x2="43.18" y2="23.705825" width="0.6096" layer="16"/>
-<wire x1="43.18" y1="23.705825" x2="43.18" y2="21.59" width="0.6096" layer="16"/>
-<wire x1="43.18" y1="21.59" x2="50.165" y2="21.59" width="0.6096" layer="16"/>
-<wire x1="50.165" y1="21.59" x2="52.705" y2="21.59" width="0.6096" layer="16"/>
-<wire x1="52.705" y1="21.59" x2="52.705" y2="24.0538" width="0.6096" layer="16"/>
-<wire x1="52.705" y1="24.0538" x2="53.975" y2="24.0538" width="0.6096" layer="16"/>
-<wire x1="53.975" y1="24.0538" x2="55.245" y2="24.0538" width="0.6096" layer="16"/>
-<wire x1="24.6888625" y1="23.705825" x2="23.4188625" y2="23.705825" width="0.6096" layer="16"/>
-<wire x1="23.4188625" y1="23.705825" x2="22.1488625" y2="23.705825" width="0.6096" layer="16"/>
-<wire x1="22.327175" y1="20.17160625" x2="22.1488625" y2="19.71491875" width="0.4064" layer="16" curve="-90"/>
-<wire x1="22.1488625" y1="19.71491875" x2="22.1488625" y2="23.705825" width="0.4064" layer="16"/>
-<wire x1="49.2125" y1="21.59" x2="50.165" y2="21.59" width="0.4064" layer="16"/>
-<polygon width="0" layer="16" isolate="0.4064" thermals="no">
-<vertex x="39.243" y="36.703"/>
-<vertex x="45.212" y="36.703"/>
-<vertex x="45.339" y="22.86"/>
-<vertex x="52.705" y="22.86"/>
-<vertex x="52.705" y="24.13"/>
-<vertex x="57.15" y="24.13"/>
-<vertex x="57.15" y="20.32"/>
-<vertex x="22.225" y="20.32"/>
-<vertex x="22.225" y="23.8125"/>
-<vertex x="39.37" y="23.8125"/>
-</polygon>
-<wire x1="45.8225" y1="24.4475" x2="43.18" y2="24.4475" width="0.4064" layer="16"/>
-<wire x1="112.9713625" y1="21.59461875" x2="111.06174375" y2="19.685" width="0.6096" layer="16"/>
-<wire x1="55.245" y1="24.0538" x2="55.4863" y2="23.8125" width="0.4064" layer="16"/>
-<wire x1="55.4863" y1="23.8125" x2="60.6425" y2="23.8125" width="0.6096" layer="16"/>
-<via x="60.6425" y="23.8125" extent="1-16" drill="0.8" diameter="1.27"/>
-<wire x1="60.6425" y1="23.8125" x2="64.77" y2="19.685" width="0.6096" layer="1"/>
-<wire x1="64.77" y1="19.685" x2="85.09" y2="19.685" width="0.6096" layer="1"/>
-<via x="85.09" y="19.685" extent="1-16" drill="0.8" diameter="1.27"/>
-<wire x1="85.09" y1="19.685" x2="111.06174375" y2="19.685" width="0.6096" layer="16"/>
-</signal>
 <signal name="N$2">
 <contactref element="Q2" pad="3"/>
@@
 <wire x1="65.19" y1="30.48" x2="61.175" y2="30.48" width="0.4064" layer="16"/>
 </signal>
+<signal name="+9V">
+<contactref element="R3" pad="2"/>
+<contactref element="R4" pad="2"/>
+<contactref element="U$3" pad="1"/>
+<contactref element="U$3" pad="3"/>
+<contactref element="U$3" pad="2"/>
+<contactref element="U$2" pad="3"/>
+<contactref element="U$2" pad="1"/>
+<contactref element="U$2" pad="2"/>
+<wire x1="52.705" y1="24.0538" x2="53.975" y2="24.0538" width="0.6096" layer="16"/>
+<wire x1="53.975" y1="24.0538" x2="55.245" y2="24.0538" width="0.6096" layer="16"/>
+<wire x1="24.6888625" y1="23.705825" x2="23.4188625" y2="23.705825" width="0.6096" layer="16"/>
+<wire x1="23.4188625" y1="23.705825" x2="22.1488625" y2="23.705825" width="0.6096" layer="16"/>
+<wire x1="22.327175" y1="20.17160625" x2="22.1488625" y2="19.71491875" width="0.4064" layer="16" curve="-90"/>
+<wire x1="22.1488625" y1="19.71491875" x2="22.1488625" y2="23.705825" width="0.4064" layer="16"/>
+<contactref element="U$1" pad="VIN"/>
+<contactref element="JP_12V" pad="1"/>
+<wire x1="43.18" y1="35.56" x2="43.18" y2="24.511" width="0.6096" layer="16"/>
+<wire x1="43.18" y1="24.511" x2="43.18" y2="24.4475" width="0.6096" layer="16"/>
+<wire x1="43.18" y1="24.4475" x2="43.18" y2="21.59" width="0.6096" layer="16"/>
+<wire x1="43.18" y1="21.59" x2="50.165" y2="21.59" width="0.6096" layer="16"/>
+<wire x1="50.165" y1="21.59" x2="52.705" y2="21.59" width="0.6096" layer="16"/>
+<wire x1="49.2125" y1="21.59" x2="50.165" y2="21.59" width="0.4064" layer="16"/>
+<wire x1="112.9713625" y1="21.59461875" x2="111.06174375" y2="19.685" width="0.6096" layer="16"/>
+<wire x1="55.4863" y1="23.8125" x2="60.6425" y2="23.8125" width="0.6096" layer="16"/>
+<via x="60.6425" y="23.8125" extent="1-16" drill="0.8" diameter="1.27"/>
+<wire x1="60.6425" y1="23.8125" x2="64.77" y2="19.685" width="0.6096" layer="1"/>
+<wire x1="64.77" y1="19.685" x2="85.09" y2="19.685" width="0.6096" layer="1"/>
+<via x="85.09" y="19.685" extent="1-16" drill="0.8" diameter="1.27"/>
+<wire x1="85.09" y1="19.685" x2="111.06174375" y2="19.685" width="0.6096" layer="16"/>
+<polygon width="0" layer="16" isolate="0.4064" thermals="no">
+<vertex x="39.243" y="36.703"/>
+<vertex x="45.212" y="36.703"/>
+<vertex x="45.339" y="22.86"/>
+<vertex x="52.705" y="22.86"/>
+<vertex x="52.705" y="24.13"/>
+<vertex x="57.15" y="24.13"/>
+<vertex x="57.15" y="20.32"/>
+<vertex x="22.225" y="20.32"/>
+<vertex x="22.225" y="23.8125"/>
+<vertex x="39.37" y="23.8125"/>
+</polygon>
+<wire x1="45.8225" y1="24.4475" x2="43.18" y2="24.4475" width="0.4064" layer="16"/>
+</signal>
 </signals>
