File: eagle/aWXIrons/main.sch (EAGLE design)
At the start: 52 parts, among them IC1_DUAL OPA336U, IC1_SINGLE OPA336U, Q1 BSN20, Q2 BSN20

Commit message: Change +12V to +9V in schematic and PCBs. Update PDFs.
Connections:
- net +12V renamed +9V
Other:
- note added: "1.2.1"
- note removed: "1.2"
